Commit message: set self collision enabled at the link level (at model level didn't seem to make any difference...)

File: soft_hand_description/model/soft_hand.gazebo.xacro (robot description, xacro)
@@ -27,4 +27,9 @@
 	</xacro:property>
 	<!-- <xacro:insert_block name="gazebo_friction_properties"/> -->
+	<!-- configure how all links will behave in gazebo (particular behavior can be set at each link as well) -->
+	<xacro:property name="gazebo_link_elements">
+		<selfCollide>true</selfCollide>
+		<xacro:insert_block name="gazebo_friction_properties"/>
+	</xacro:property>
 	<xacro:property name="gazebo_other_properties">
 		<!-- <material>value</material> -->
@@ -76,5 +81,5 @@
 				</plugin>
 			</sensor>
-			<xacro:insert_block name="gazebo_friction_properties"/>
+			<xacro:insert_block name="gazebo_link_elements"/>
 		</gazebo>
 		<gazebo reference="${name}_thumb_knuckle_link">
@@ -95,5 +100,5 @@
 				</plugin>
 			</sensor>
-			<xacro:insert_block name="gazebo_friction_properties"/>
+			<xacro:insert_block name="gazebo_link_elements"/>
 		</gazebo>
 		<gazebo reference="${name}_thumb_proximal_link">
@@ -114,5 +119,5 @@
 				</plugin>
 			</sensor>
-			<xacro:insert_block name="gazebo_friction_properties"/>
+			<xacro:insert_block name="gazebo_link_elements"/>
 		</gazebo>
 		<gazebo reference="${name}_thumb_distal_link">
@@ -133,5 +138,5 @@
 				</plugin>
 			</sensor>
-			<xacro:insert_block name="gazebo_friction_properties"/>
+			<xacro:insert_block name="gazebo_link_elements"/>
 		</gazebo>
 		<gazebo reference="${name}_index_knuckle_link">
@@ -152,5 +157,5 @@
 				</plugin>
 			</sensor>
-			<xacro:insert_block name="gazebo_friction_properties"/>
+			<xacro:insert_block name="gazebo_link_elements"/>
 		</gazebo>
 		<gazebo reference="${name}_index_proximal_link">
@@ -171,5 +176,5 @@
 				</plugin>
 			</sensor>
-			<xacro:insert_block name="gazebo_friction_properties"/>
+			<xacro:insert_block name="gazebo_link_elements"/>
 		</gazebo>
 		<gazebo reference="${name}_index_middle_link">
@@ -190,5 +195,5 @@
 				</plugin>
 			</sensor>
-			<xacro:insert_block name="gazebo_friction_properties"/>
+			<xacro:insert_block name="gazebo_link_elements"/>
 		</gazebo>
 		<gazebo reference="${name}_index_distal_link">
@@ -209,5 +214,5 @@
 				</plugin>
 			</sensor>
-			<xacro:insert_block name="gazebo_friction_properties"/>
+			<xacro:insert_block name="gazebo_link_elements"/>
 		</gazebo>
 		<gazebo reference="${name}_middle_knuckle_link">
@@ -228,5 +233,5 @@
 				</plugin>
 			</sensor>
-			<xacro:insert_block name="gazebo_friction_properties"/>
+			<xacro:insert_block name="gazebo_link_elements"/>
 		</gazebo>
 		<gazebo reference="${name}_middle_proximal_link">
@@ -247,5 +252,5 @@
 				</plugin>
 			</sensor>
-			<xacro:insert_block name="gazebo_friction_properties"/>
+			<xacro:insert_block name="gazebo_link_elements"/>
 		</gazebo>
 		<gazebo reference="${name}_middle_middle_link">
@@ -266,5 +271,5 @@
 				</plugin>
 			</sensor>
-			<xacro:insert_block name="gazebo_friction_properties"/>
+			<xacro:insert_block name="gazebo_link_elements"/>
 		</gazebo>
 		<gazebo reference="${name}_middle_distal_link">
@@ -285,5 +290,5 @@
 				</plugin>
 			</sensor>
-			<xacro:insert_block name="gazebo_friction_properties"/>
+			<xacro:insert_block name="gazebo_link_elements"/>
 		</gazebo>
 		<gazebo reference="${name}_ring_knuckle_link">
@@ -304,5 +309,5 @@
 				</plugin>
 			</sensor>
-			<xacro:insert_block name="gazebo_friction_properties"/>
+			<xacro:insert_block name="gazebo_link_elements"/>
 		</gazebo>
 		<gazebo reference="${name}_ring_proximal_link">
@@ -323,5 +328,5 @@
 				</plugin>
 			</sensor>
-			<xacro:insert_block name="gazebo_friction_properties"/>
+			<xacro:insert_block name="gazebo_link_elements"/>
 		</gazebo>
 		<gazebo reference="${name}_ring_middle_link">
@@ -342,5 +347,5 @@
 				</plugin>
 			</sensor>
-			<xacro:insert_block name="gazebo_friction_properties"/>
+			<xacro:insert_block name="gazebo_link_elements"/>
 		</gazebo>
 		<gazebo reference="${name}_ring_distal_link">
@@ -361,5 +366,5 @@
 				</plugin>
 			</sensor>
-			<xacro:insert_block name="gazebo_friction_properties"/>
+			<xacro:insert_block name="gazebo_link_elements"/>
 		</gazebo>
 		<gazebo reference="${name}_little_knuckle_link">
@@ -380,5 +385,5 @@
 				</plugin>
 			</sensor>
-			<xacro:insert_block name="gazebo_friction_properties"/>
+			<xacro:insert_block name="gazebo_link_elements"/>
 		</gazebo>
 		<gazebo reference="${name}_little_proximal_link">
@@ -399,5 +404,5 @@
 				</plugin>
 			</sensor>
-			<xacro:insert_block name="gazebo_friction_properties"/>
+			<xacro:insert_block name="gazebo_link_elements"/>
 		</gazebo>
 		<gazebo reference="${name}_little_middle_link">
@@ -418,5 +423,5 @@
 				</plugin>
 			</sensor>
-			<xacro:insert_block name="gazebo_friction_properties"/>
+			<xacro:insert_block name="gazebo_link_elements"/>
 		</gazebo>
 		<gazebo reference="${name}_little_distal_link">
@@ -437,5 +442,5 @@
 				</plugin>
 			</sensor>
-			<xacro:insert_block name="gazebo_friction_properties"/>
+			<xacro:insert_block name="gazebo_link_elements"/>
 		</gazebo>
 		<!-- JOINTS -->

Commit message: added bitmask which should be useful in gazebo6. NOT tested.

File: soft_hand_description/model/soft_hand.gazebo.xacro (robot description, xacro)
@@ -38,4 +38,11 @@
 	</xacro:property>
 	<!-- <xacro:insert_block name="gazebo_other_properties"/> -->
+	<xacro:macro name="collideBitmask" params="hex_collision">
+		<surface>
+			<contact>
+				<collide_bitmask>${hex_collision}</collide_bitmask>
+			</contact>
+		</surface>
+	</xacro:macro>
 	<xacro:macro name="soft_hand_gazebo" params="name withAdaptiveTransmission useMimicTag">
 		<!-- PLUGINS -->
@@ -444,4 +451,66 @@
 			<xacro:insert_block name="gazebo_link_elements"/>
 		</gazebo>
+		<!-- COLLISIONS -->
+		<!-- values generated using a Matlab script to make sure no consecutive links will collide, and no knuckle will collide with the palm -->
+		<gazebo reference="${name}_palm_link_collision">
+			<xacro:collideBitmask hex_collision="0x4925"/>
+		</gazebo>
+		<gazebo reference="${name}_thumb_knuckle_link_collision">
+			<xacro:collideBitmask hex_collision="0x2492"/>
+		</gazebo>
+		<gazebo reference="${name}_thumb_proximal_link_collision">
+			<xacro:collideBitmask hex_collision="0x0009"/>
+		</gazebo>
+		<gazebo reference="${name}_thumb_distal_link_collision">
+			<xacro:collideBitmask hex_collision="0x0006"/>
+		</gazebo>
+		<gazebo reference="${name}_index_knuckle_link_collision">
+			<xacro:collideBitmask hex_collision="0x24CA"/>
+		</gazebo>
+		<gazebo reference="${name}_index_proximal_link_collision">
+			<xacro:collideBitmask hex_collision="0x0015"/>
+		</gazebo>
+		<gazebo reference="${name}_index_middle_link_collision">
+			<xacro:collideBitmask hex_collision="0x002A"/>
+		</gazebo>
+		<gazebo reference="${name}_index_distal_link_collision">
+			<xacro:collideBitmask hex_collision="0x0055"/>
+		</gazebo>
+		<gazebo reference="${name}_middle_knuckle_link_collision">
+			<xacro:collideBitmask hex_collision="0x265A"/>
+		</gazebo>
+		<gazebo reference="${name}_middle_proximal_link_collision">
+			<xacro:collideBitmask hex_collision="0x00A5"/>
+		</gazebo>
+		<gazebo reference="${name}_middle_middle_link_collision">
+			<xacro:collideBitmask hex_collision="0x015A"/>
+		</gazebo>
+		<gazebo reference="${name}_middle_distal_link_collision">
+			<xacro:collideBitmask hex_collision="0x02A5"/>
+		</gazebo>
+		<gazebo reference="${name}_ring_knuckle_link_collision">
+			<xacro:collideBitmask hex_collision="0x32DA"/>
+		</gazebo>
+		<gazebo reference="${name}_ring_proximal_link_collision">
+			<xacro:collideBitmask hex_collision="0x0525"/>
+		</gazebo>
+		<gazebo reference="${name}_ring_middle_link_collision">
+			<xacro:collideBitmask hex_collision="0x0ADA"/>
+		</gazebo>
+		<gazebo reference="${name}_ring_distal_link_collision">
+			<xacro:collideBitmask hex_collision="0x1525"/>
+		</gazebo>
+		<gazebo reference="${name}_little_knuckle_link_collision">
+			<xacro:collideBitmask hex_collision="0x96DA"/>
+		</gazebo>
+		<gazebo reference="${name}_little_proximal_link_collision">
+			<xacro:collideBitmask hex_collision="0x2925"/>
+		</gazebo>
+		<gazebo reference="${name}_little_middle_link_collision">
+			<xacro:collideBitmask hex_collision="0x56DA"/>
+		</gazebo>
+		<gazebo reference="${name}_little_distal_link_collision">
+			<xacro:collideBitmask hex_collision="0xA925"/>
+		</gazebo>
 		<!-- JOINTS -->
 		<gazebo reference="${name}_thumb_abd_joint">

Commit message: tested collide bitmasks, now they actually work using Gazebo6

File: soft_hand_description/model/soft_hand.gazebo.xacro (robot description, xacro)
@@ -89,4 +89,7 @@
 			</sensor>
 			<xacro:insert_block name="gazebo_link_elements"/>
+			<collision>
+				<xacro:collideBitmask hex_collision="0x4925"/>
+			</collision>
 		</gazebo>
 		<gazebo reference="${name}_thumb_knuckle_link">
@@ -108,4 +111,7 @@
 			</sensor>
 			<xacro:insert_block name="gazebo_link_elements"/>
+			<collision>
+				<xacro:collideBitmask hex_collision="0x2492"/>
+			</collision>
 		</gazebo>
 		<gazebo reference="${name}_thumb_proximal_link">
@@ -127,4 +133,7 @@
 			</sensor>
 			<xacro:insert_block name="gazebo_link_elements"/>
+			<collision>
+				<xacro:collideBitmask hex_collision="0x0009"/>
+			</collision>
 		</gazebo>
 		<gazebo reference="${name}_thumb_distal_link">
@@ -146,4 +155,7 @@
 			</sensor>
 			<xacro:insert_block name="gazebo_link_elements"/>
+			<collision>
+				<xacro:collideBitmask hex_collision="0x0006"/>
+			</collision>
 		</gazebo>
 		<gazebo reference="${name}_index_knuckle_link">
@@ -165,4 +177,7 @@
 			</sensor>
 			<xacro:insert_block name="gazebo_link_elements"/>
+			<collision>
+				<xacro:collideBitmask hex_collision="0x24CA"/>
+			</collision>
 		</gazebo>
 		<gazebo reference="${name}_index_proximal_link">
@@ -184,4 +199,7 @@
 			</sensor>
 			<xacro:insert_block name="gazebo_link_elements"/>
+			<collision>
+				<xacro:collideBitmask hex_collision="0x0015"/>
+			</collision>
 		</gazebo>
 		<gazebo reference="${name}_index_middle_link">
@@ -203,4 +221,7 @@
 			</sensor>
 			<xacro:insert_block name="gazebo_link_elements"/>
+			<collision>
+				<xacro:collideBitmask hex_collision="0x002A"/>
+			</collision>
 		</gazebo>
 		<gazebo reference="${name}_index_distal_link">
@@ -222,4 +243,7 @@
 			</sensor>
 			<xacro:insert_block name="gazebo_link_elements"/>
+			<collision>
+				<xacro:collideBitmask hex_collision="0x0055"/>
+			</collision>
 		</gazebo>
 		<gazebo reference="${name}_middle_knuckle_link">
@@ -241,4 +265,7 @@
 			</sensor>
 			<xacro:insert_block name="gazebo_link_elements"/>
+			<collision>
+				<xacro:collideBitmask hex_collision="0x265A"/>
+			</collision>
 		</gazebo>
 		<gazebo reference="${name}_middle_proximal_link">
@@ -260,4 +287,7 @@
 			</sensor>
 			<xacro:insert_block name="gazebo_link_elements"/>
+			<collision>
+				<xacro:collideBitmask hex_collision="0x00A5"/>
+			</collision>
 		</gazebo>
 		<gazebo reference="${name}_middle_middle_link">
@@ -279,4 +309,7 @@
 			</sensor>
 			<xacro:insert_block name="gazebo_link_elements"/>
+			<collision>
+				<xacro:collideBitmask hex_collision="0x015A"/>
+			</collision>
 		</gazebo>
 		<gazebo reference="${name}_middle_distal_link">
@@ -298,4 +331,7 @@
 			</sensor>
 			<xacro:insert_block name="gazebo_link_elements"/>
+			<collision>
+				<xacro:collideBitmask hex_collision="0x02A5"/>
+			</collision>
 		</gazebo>
 		<gazebo reference="${name}_ring_knuckle_link">
@@ -317,4 +353,7 @@
 			</sensor>
 			<xacro:insert_block name="gazebo_link_elements"/>
+			<collision>
+				<xacro:collideBitmask hex_collision="0x32DA"/>
+			</collision>
 		</gazebo>
 		<gazebo reference="${name}_ring_proximal_link">
@@ -336,4 +375,7 @@
 			</sensor>
 			<xacro:insert_block name="gazebo_link_elements"/>
+			<collision>
+				<xacro:collideBitmask hex_collision="0x0525"/>
+			</collision>
 		</gazebo>
 		<gazebo reference="${name}_ring_middle_link">
@@ -355,4 +397,7 @@
 			</sensor>
 			<xacro:insert_block name="gazebo_link_elements"/>
+			<collision>
+				<xacro:collideBitmask hex_collision="0x0ADA"/>
+			</collision>
 		</gazebo>
 		<gazebo reference="${name}_ring_distal_link">
@@ -374,4 +419,7 @@
 			</sensor>
 			<xacro:insert_block name="gazebo_link_elements"/>
+			<collision>
+				<xacro:collideBitmask hex_collision="0x1525"/>
+			</collision>
 		</gazebo>
 		<gazebo reference="${name}_little_knuckle_link">
@@ -393,4 +441,7 @@
 			</sensor>
 			<xacro:insert_block name="gazebo_link_elements"/>
+			<collision>
+				<xacro:collideBitmask hex_collision="0x96DA"/>
+			</collision>
 		</gazebo>
 		<gazebo reference="${name}_little_proximal_link">
@@ -412,4 +463,7 @@
 			</sensor>
 			<xacro:insert_block name="gazebo_link_elements"/>
+			<collision>
+				<xacro:collideBitmask hex_collision="0x2925"/>
+			</collision>
 		</gazebo>
 		<gazebo reference="${name}_little_middle_link">
@@ -431,4 +485,7 @@
 			</sensor>
 			<xacro:insert_block name="gazebo_link_elements"/>
+			<collision>
+				<xacro:collideBitmask hex_collision="0x56DA"/>
+			</collision>
 		</gazebo>
 		<gazebo reference="${name}_little_distal_link">
@@ -450,66 +507,7 @@
 			</sensor>
 			<xacro:insert_block name="gazebo_link_elements"/>
-		</gazebo>
-		<!-- COLLISIONS -->
-		<!-- values generated using a Matlab script to make sure no consecutive links will collide, and no knuckle will collide with the palm -->
-		<gazebo reference="${name}_palm_link_collision">
-			<xacro:collideBitmask hex_collision="0x4925"/>
-		</gazebo>
-		<gazebo reference="${name}_thumb_knuckle_link_collision">
-			<xacro:collideBitmask hex_collision="0x2492"/>
-		</gazebo>
-		<gazebo reference="${name}_thumb_proximal_link_collision">
-			<xacro:collideBitmask hex_collision="0x0009"/>
-		</gazebo>
-		<gazebo reference="${name}_thumb_distal_link_collision">
-			<xacro:collideBitmask hex_collision="0x0006"/>
-		</gazebo>
-		<gazebo reference="${name}_index_knuckle_link_collision">
-			<xacro:collideBitmask hex_collision="0x24CA"/>
-		</gazebo>
-		<gazebo reference="${name}_index_proximal_link_collision">
-			<xacro:collideBitmask hex_collision="0x0015"/>
-		</gazebo>
-		<gazebo reference="${name}_index_middle_link_collision">
-			<xacro:collideBitmask hex_collision="0x002A"/>
-		</gazebo>
-		<gazebo reference="${name}_index_distal_link_collision">
-			<xacro:collideBitmask hex_collision="0x0055"/>
-		</gazebo>
-		<gazebo reference="${name}_middle_knuckle_link_collision">
-			<xacro:collideBitmask hex_collision="0x265A"/>
-		</gazebo>
-		<gazebo reference="${name}_middle_proximal_link_collision">
-			<xacro:collideBitmask hex_collision="0x00A5"/>
-		</gazebo>
-		<gazebo reference="${name}_middle_middle_link_collision">
-			<xacro:collideBitmask hex_collision="0x015A"/>
-		</gazebo>
-		<gazebo reference="${name}_middle_distal_link_collision">
-			<xacro:collideBitmask hex_collision="0x02A5"/>
-		</gazebo>
-		<gazebo reference="${name}_ring_knuckle_link_collision">
-			<xacro:collideBitmask hex_collision="0x32DA"/>
-		</gazebo>
-		<gazebo reference="${name}_ring_proximal_link_collision">
-			<xacro:collideBitmask hex_collision="0x0525"/>
-		</gazebo>
-		<gazebo reference="${name}_ring_middle_link_collision">
-			<xacro:collideBitmask hex_collision="0x0ADA"/>
-		</gazebo>
-		<gazebo reference="${name}_ring_distal_link_collision">
-			<xacro:collideBitmask hex_collision="0x1525"/>
-		</gazebo>
-		<gazebo reference="${name}_little_knuckle_link_collision">
-			<xacro:collideBitmask hex_collision="0x96DA"/>
-		</gazebo>
-		<gazebo reference="${name}_little_proximal_link_collision">
-			<xacro:collideBitmask hex_collision="0x2925"/>
-		</gazebo>
-		<gazebo reference="${name}_little_middle_link_collision">
-			<xacro:collideBitmask hex_collision="0x56DA"/>
-		</gazebo>
-		<gazebo reference="${name}_little_distal_link_collision">
-			<xacro:collideBitmask hex_collision="0xA925"/>
+			<collision>
+				<xacro:collideBitmask hex_collision="0xA925"/>
+			</collision>
 		</gazebo>
 		<!-- JOINTS -->

Commit message: adapted selfCollide properties and collision bitmasks to work better (there were collisions between proximal phalanxes and the palm)

File: soft_hand_description/model/soft_hand.gazebo.xacro (robot description, xacro)
@@ -32,4 +32,8 @@
 		<xacro:insert_block name="gazebo_friction_properties"/>
 	</xacro:property>
+	<xacro:property name="gazebo_nonSelfCollide_link_elements">
+		<selfCollide>false</selfCollide>
+		<xacro:insert_block name="gazebo_friction_properties"/>
+	</xacro:property>
 	<xacro:property name="gazebo_other_properties">
 		<!-- <material>value</material> -->
@@ -90,5 +94,5 @@
 			<xacro:insert_block name="gazebo_link_elements"/>
 			<collision>
-				<xacro:collideBitmask hex_collision="0x4925"/>
+				<xacro:collideBitmask hex_collision="0x49250"/>
 			</collision>
 		</gazebo>
@@ -110,7 +114,8 @@
 				</plugin>
 			</sensor>
-			<xacro:insert_block name="gazebo_link_elements"/>
-			<collision>
-				<xacro:collideBitmask hex_collision="0x2492"/>
+			<xacro:insert_block name="gazebo_nonSelfCollide_link_elements"/>
+			<collision>
+				<!-- <xacro:collideBitmask hex_collision="0x24920"/> -->
+				<xacro:collideBitmask hex_collision="0x1"/>
 			</collision>
 		</gazebo>
@@ -134,5 +139,5 @@
 			<xacro:insert_block name="gazebo_link_elements"/>
 			<collision>
-				<xacro:collideBitmask hex_collision="0x0009"/>
+				<xacro:collideBitmask hex_collision="0x00090"/>
 			</collision>
 		</gazebo>
@@ -156,5 +161,5 @@
 			<xacro:insert_block name="gazebo_link_elements"/>
 			<collision>
-				<xacro:collideBitmask hex_collision="0x0006"/>
+				<xacro:collideBitmask hex_collision="0x00060"/>
 			</collision>
 		</gazebo>
@@ -176,7 +181,8 @@
 				</plugin>
 			</sensor>
-			<xacro:insert_block name="gazebo_link_elements"/>
-			<collision>
-				<xacro:collideBitmask hex_collision="0x24CA"/>
+			<xacro:insert_block name="gazebo_nonSelfCollide_link_elements"/>
+			<collision>
+				<!-- <xacro:collideBitmask hex_collision="0x24CA0"/> -->
+				<xacro:collideBitmask hex_collision="0x1"/>
 			</collision>
 		</gazebo>
@@ -198,7 +204,8 @@
 				</plugin>
 			</sensor>
-			<xacro:insert_block name="gazebo_link_elements"/>
-			<collision>
-				<xacro:collideBitmask hex_collision="0x0015"/>
+			<xacro:insert_block name="gazebo_nonSelfCollide_link_elements"/>
+			<collision>
+				<!-- <xacro:collideBitmask hex_collision="0x00150"/> -->
+				<xacro:collideBitmask hex_collision="0x2"/>
 			</collision>
 		</gazebo>
@@ -222,5 +229,5 @@
 			<xacro:insert_block name="gazebo_link_elements"/>
 			<collision>
-				<xacro:collideBitmask hex_collision="0x002A"/>
+				<xacro:collideBitmask hex_collision="0x002A0"/>
 			</collision>
 		</gazebo>
@@ -244,5 +251,5 @@
 			<xacro:insert_block name="gazebo_link_elements"/>
 			<collision>
-				<xacro:collideBitmask hex_collision="0x0055"/>
+				<xacro:collideBitmask hex_collision="0x00550"/>
 			</collision>
 		</gazebo>
@@ -264,7 +271,8 @@
 				</plugin>
 			</sensor>
-			<xacro:insert_block name="gazebo_link_elements"/>
-			<collision>
-				<xacro:collideBitmask hex_collision="0x265A"/>
+			<xacro:insert_block name="gazebo_nonSelfCollide_link_elements"/>
+			<collision>
+				<!-- <xacro:collideBitmask hex_collision="0x265A0"/> -->
+				<xacro:collideBitmask hex_collision="0x1"/>
 			</collision>
 		</gazebo>
@@ -286,7 +294,8 @@
 				</plugin>
 			</sensor>
-			<xacro:insert_block name="gazebo_link_elements"/>
-			<collision>
-				<xacro:collideBitmask hex_collision="0x00A5"/>
+			<xacro:insert_block name="gazebo_nonSelfCollide_link_elements"/>
+			<collision>
+				<!-- <xacro:collideBitmask hex_collision="0x00A50"/> -->
+				<xacro:collideBitmask hex_collision="0x2"/>
 			</collision>
 		</gazebo>
@@ -310,5 +319,5 @@
 			<xacro:insert_block name="gazebo_link_elements"/>
 			<collision>
-				<xacro:collideBitmask hex_collision="0x015A"/>
+				<xacro:collideBitmask hex_collision="0x015A0"/>
 			</collision>
 		</gazebo>
@@ -332,5 +341,5 @@
 			<xacro:insert_block name="gazebo_link_elements"/>
 			<collision>
-				<xacro:collideBitmask hex_collision="0x02A5"/>
+				<xacro:collideBitmask hex_collision="0x02A50"/>
 			</collision>
 		</gazebo>
@@ -352,7 +361,8 @@
 				</plugin>
 			</sensor>
-			<xacro:insert_block name="gazebo_link_elements"/>
-			<collision>
-				<xacro:collideBitmask hex_collision="0x32DA"/>
+			<xacro:insert_block name="gazebo_nonSelfCollide_link_elements"/>
+			<collision>
+				<!-- <xacro:collideBitmask hex_collision="0x32DA0"/> -->
+				<xacro:collideBitmask hex_collision="0x1"/>
 			</collision>
 		</gazebo>
@@ -374,7 +384,8 @@
 				</plugin>
 			</sensor>
-			<xacro:insert_block name="gazebo_link_elements"/>
-			<collision>
-				<xacro:collideBitmask hex_collision="0x0525"/>
+			<xacro:insert_block name="gazebo_nonSelfCollide_link_elements"/>
+			<collision>
+				<!-- <xacro:collideBitmask hex_collision="0x05250"/> -->
+				<xacro:collideBitmask hex_collision="0x2"/>
 			</collision>
 		</gazebo>
@@ -398,5 +409,5 @@
 			<xacro:insert_block name="gazebo_link_elements"/>
 			<collision>
-				<xacro:collideBitmask hex_collision="0x0ADA"/>
+				<xacro:collideBitmask hex_collision="0x0ADA0"/>
 			</collision>
 		</gazebo>
@@ -420,5 +431,5 @@
 			<xacro:insert_block name="gazebo_link_elements"/>
 			<collision>
-				<xacro:collideBitmask hex_collision="0x1525"/>
+				<xacro:collideBitmask hex_collision="0x15250"/>
 			</collision>
 		</gazebo>
@@ -440,7 +451,8 @@
 				</plugin>
 			</sensor>
-			<xacro:insert_block name="gazebo_link_elements"/>
-			<collision>
-				<xacro:collideBitmask hex_collision="0x96DA"/>
+			<xacro:insert_block name="gazebo_nonSelfCollide_link_elements"/>
+			<collision>
+				<!-- <xacro:collideBitmask hex_collision="0x96DA0"/> -->
+				<xacro:collideBitmask hex_collision="0x1"/>
 			</collision>
 		</gazebo>
@@ -462,7 +474,8 @@
 				</plugin>
 			</sensor>
-			<xacro:insert_block name="gazebo_link_elements"/>
-			<collision>
-				<xacro:collideBitmask hex_collision="0x2925"/>
+			<xacro:insert_block name="gazebo_nonSelfCollide_link_elements"/>
+			<collision>
+				<!-- <xacro:collideBitmask hex_collision="0x29250"/> -->
+				<xacro:collideBitmask hex_collision="0x2"/>
 			</collision>
 		</gazebo>
@@ -486,5 +499,5 @@
 			<xacro:insert_block name="gazebo_link_elements"/>
 			<collision>
-				<xacro:collideBitmask hex_collision="0x56DA"/>
+				<xacro:collideBitmask hex_collision="0x56DA0"/>
 			</collision>
 		</gazebo>
@@ -508,5 +521,5 @@
 			<xacro:insert_block name="gazebo_link_elements"/>
 			<collision>
-				<xacro:collideBitmask hex_collision="0xA925"/>
+				<xacro:collideBitmask hex_collision="0xA9250"/>
 			</collision>
 		</gazebo>
